File: VCU/Hardware/VCU2.0/VCU2.0.kicad_sch (KiCad schematic)
At the start: 4 parts

Commit message: mimi
Other:
- sheet IO renamed e
Changed lines of the file:
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@@
 		)
 		(fill
-			(color 0 0 0 0.0000)
+			(color 128 255 128 1.0000)
 		)
 		(property "Sheetname" "PowerMGMT"
@@
 		)
 		(fill
-			(color 0 0 0 0.0000)
+			(color 128 255 128 1.0000)
 		)
 		(property "Sheetname" "Connector"
@@
 				)
 				(justify left top)
+			)
+		)
+		(property "Field2" ""
+			(at 175.26 48.895 0)
+			(effects
+				(font
+					(size 1.27 1.27)
+				)
+				(hide yes)
 			)
 		)
@@
 		)
 		(fill
-			(color 0 0 0 0.0000)
+			(color 128 255 128 1.0000)
 		)
 		(property "Sheetname" "Supply"
@@
 		)
 		(fill
-			(color 0 0 0 0.0000)
+			(color 128 255 128 1.0000)
 		)
 		(property "Sheetname" "esp32S3"
@@
 		)
 		(fill
-			(color 0 0 0 0.0000)
-		)
-		(property "Sheetname" "IO"
+			(color 128 255 128 1.0000)
+		)
+		(property "Sheetname" "e"
 			(at 140.97 48.1834 0)
 			(effects
