File: Speedometer_KiCAD/Hardware/Speedometer_Tech/110_ESP32s3.kicad_sch (KiCad schematic)
At the start: 26 parts, among them P1100 TYPEC-300D-BCP16H100, P1101 5-146130-2, P1102 M20-8770442R, P1103 5-146130-2, P1104 HTSS-105-01-L-DV, Q1103 DTC123JET1G, Q1104 DTC123JET1G, U1100 ESP32WroomS3

Commit message: we got speeddo
Parts:
- S1100, S1101, S1103, S1104: value (none) -> ~
Changed lines of the file:
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@@
 	(label "USB D+"
 		(at 220.98 80.4672 0)
+		(fields_autoplaced yes)
 		(effects
 			(font
@@
 	(label "MISO"
 		(at 71.12 88.0872 0)
+		(fields_autoplaced yes)
 		(effects
 			(font
@@
 	(label "EN"
 		(at 177.8 133.8072 0)
+		(fields_autoplaced yes)
 		(effects
 			(font
@@
 	(label "USB D-"
 		(at 203.2 70.3072 0)
+		(fields_autoplaced yes)
 		(effects
 			(font
@@
 	(label "SDA"
 		(at 149.86 171.9072 0)
+		(fields_autoplaced yes)
 		(effects
 			(font
@@
 	(label "USB D-"
 		(at 152.4 70.3072 0)
+		(fields_autoplaced yes)
 		(effects
 			(font
@@
 	(label "EN"
 		(at 198.12 136.3472 0)
+		(fields_autoplaced yes)
 		(effects
 			(font
@@
 	(label "USB D+"
 		(at 111.76 83.0072 0)
+		(fields_autoplaced yes)
 		(effects
 			(font
@@
 	(label "MTCK"
 		(at 111.76 98.2472 0)
+		(fields_autoplaced yes)
 		(effects
 			(font
@@
 	(label "SCK"
 		(at 71.12 85.5472 0)
+		(fields_autoplaced yes)
 		(effects
 			(font
@@
 	(label "MTMS"
 		(at 111.76 105.8672 0)
+		(fields_autoplaced yes)
 		(effects
 			(font
@@
 	(label "EN"
 		(at 215.9 174.4472 0)
+		(fields_autoplaced yes)
 		(effects
 			(font
@@
 	(label "SCL"
 		(at 73.66 80.4672 0)
+		(fields_autoplaced yes)
 		(effects
 			(font
@@
 	(label "TX"
 		(at 73.66 70.3072 0)
+		(fields_autoplaced yes)
 		(effects
 			(font
@@
 	(label "USB D-"
 		(at 111.76 80.4672 0)
+		(fields_autoplaced yes)
 		(effects
 			(font
@@
 	(label "RX"
 		(at 149.86 133.8072 0)
+		(fields_autoplaced yes)
 		(effects
 			(font
@@
 	(label "Q1"
 		(at 88.9 156.6672 90)
+		(fields_autoplaced yes)
 		(effects
 			(font
@@
 	(label "USB D+"
 		(at 152.4 67.7672 0)
+		(fields_autoplaced yes)
 		(effects
 			(font
@@
 	(label "RX"
 		(at 198.12 133.8072 0)
+		(fields_autoplaced yes)
 		(effects
 			(font
@@
 	(label "USB D+"
 		(at 203.2 67.7672 0)
+		(fields_autoplaced yes)
 		(effects
 			(font
@@
 	(label "MTCK"
 		(at 215.9 166.8272 0)
+		(fields_autoplaced yes)
 		(effects
 			(font
@@
 	(label "TX"
 		(at 177.8 131.2672 0)
+		(fields_autoplaced yes)
 		(effects
 			(font
@@
 	(label "MTDO"
 		(at 111.76 100.7872 0)
+		(fields_autoplaced yes)
 		(effects
 			(font
@@
 	(label "MOSI"
 		(at 71.12 90.6272 0)
+		(fields_autoplaced yes)
 		(effects
 			(font
@@
 	(label "USB D-"
 		(at 220.98 67.7672 0)
+		(fields_autoplaced yes)
 		(effects
 			(font
@@
 	(label "RX"
 		(at 73.66 67.7672 0)
+		(fields_autoplaced yes)
 		(effects
 			(font
@@
 	(label "CS"
 		(at 71.12 93.1672 0)
+		(fields_autoplaced yes)
 		(effects
 			(font
@@
 	(label "MTDI"
 		(at 215.9 171.9072 0)
+		(fields_autoplaced yes)
 		(effects
 			(font
@@
 	(label "TX"
 		(at 198.12 131.2672 0)
+		(fields_autoplaced yes)
 		(effects
 			(font
@@
 	(label "SDA"
 		(at 73.66 77.9272 0)
+		(fields_autoplaced yes)
 		(effects
 			(font
@@
 	(label "EN"
 		(at 63.5 57.6072 0)
+		(fields_autoplaced yes)
 		(effects
 			(font
@@
 	(label "MTMS"
 		(at 215.9 164.2872 0)
+		(fields_autoplaced yes)
 		(effects
 			(font
@@
 	(label "MTDO"
 		(at 215.9 169.3672 0)
+		(fields_autoplaced yes)
 		(effects
 			(font
@@
 	(label "MTDI"
 		(at 111.76 103.3272 0)
+		(fields_autoplaced yes)
 		(effects
 			(font
@@
 	(label "SCL"
 		(at 149.86 174.4472 0)
+		(fields_autoplaced yes)
 		(effects
 			(font
@@
 			)
 		)
-		(property "Value" ""
+		(property "Value" "~"
 			(at 109.982 166.5732 0)
 			(effects
@@
 			)
 		)
-		(property "Value" ""
+		(property "Value" "~"
 			(at 32.766 76.1492 0)
 			(effects
@@
 			)
 		)
-		(property "Value" ""
+		(property "Value" "~"
 			(at 48.006 88.8492 0)
 			(effects
@@
 			)
 		)
-		(property "Value" ""
+		(property "Value" "~"
 			(at 56.642 166.5732 0)
 			(effects
