File: Speedometer_KiCAD/Hardware/Speedometer_Tech/60_Inkremental.kicad_sch (KiCad schematic)
At the start: 2 parts

Commit message: we got speeddo
Parts:
- S600: value (none) -> ~
Changed lines of the file:
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@@
 			)
 		)
-		(property "Value" ""
+		(property "Value" "~"
 			(at 159.766 165.6842 0)
 			(effects
