File: Speedometer/Speedometer_KiCAD_RevB/Hardware/Speedometer_Tech/Speedometer_Tech.kicad_pcb (KiCad board)
At the start: 4 copper layers, 309.2 x 103.7 mm, 246 parts, among them J800 CTB9302/9, J801 CTB9302/9, J900 CTB9302/2, P001 3P-SMD/THT, P1100 TYPEC-300D-BCP16H100, P1101 5-146130-2, P1102 M20-8770442R, P1103 5-146130-2, P1104 HTSS-105-01-L-DV, Q1103 DTC123JET1G, Q1104 DTC123JET1G, U100 TLC59108IPWR, U1000 TPS51385, U101 TLC59108IPWR, U102 TLC59108IPWR, U1020 TPS51385, U110 TLC59108IPWR, U1100 ESP32WroomS3, U111 TLC59108IPWR, U204 WS2812B-4020_2, U205 WS2812B-4020_2, U206 WS2812B-4020_2, U207 WS2812B-4020_2, U208 WS2812B-4020_2, U209 WS2812B-4020_2, U210 WS2812B-4020_2, U211 WS2812B-4020_2, U212 WS2812B-4020_2, U213 WS2812B-4020_2, U214 WS2812B-4020_2, U215 WS2812B-4020_2, U216 WS2812B-4020_2, U217 WS2812B-4020_2, U218 WS2812B-4020_2, U219 WS2812B-4020_2, U220 WS2812B-4020_2, U221 WS2812B-4020_2, U222 WS2812B-4020_2, U223 WS2812B-4020_2, U300 WS2812B-4020_2, U301 WS2812B-4020_2, U302 WS2812B-4020_2, U303 WS2812B-4020_2, U304 WS2812B-4020_2, U305 WS2812B-4020_2, U306 WS2812B-4020_2, U307 WS2812B-4020_2, U310 WS2812B-4020_2, U311 WS2812B-4020_2, U312 WS2812B-4020_2, U313 WS2812B-4020_2, U314 WS2812B-4020_2, U320 WS2812B-4020_2, U321 WS2812B-4020_2, U322 WS2812B-4020_2, U323 WS2812B-4020_2, U400 WS2812B-4020_2, U401 WS2812B-4020_2, U402 WS2812B-4020_2, U403 WS2812B-4020_2, U404 WS2812B-4020_2, U405 WS2812B-4020_2, U406 WS2812B-4020_2, U407 WS2812B-4020_2, U410 WS2812B-4020_2, U411 WS2812B-4020_2, U412 WS2812B-4020_2, U413 WS2812B-4020_2, U414 WS2812B-4020_2, U420 WS2812B-4020_2, U421 WS2812B-4020_2, U422 WS2812B-4020_2, U423 WS2812B-4020_2, U424 WS2812B-4020_2, U510 TLC59108IPWR, U511 TLC59108IPWR, U512 TLC59108IPWR, U513 TLC59108IPWR, U514 TLC59108IPWR, U515 TLC59108IPWR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

Commit message: updated troq display with new neopixel
Parts:
- removed C1001, C1002, C1003, C1021, C1022, C1023: 47uF/25V, Vault:FP-C3216-160-0_2-MFG
- removed C1004, C1006, C1024, C1026: 0.1uF/50V, Vault:CAPC2013X135X45ML10T25
- removed C1005, C1025: 1uF/10V, Vault:FP-C0603-CG-MFG
- removed C1007, C1027: 22pF/16V, Vault:FP-C0603C-CF-MFG
- removed C1008, C1009, C1010, C1011, C1028, C1029, C1030, C1031: 22uF/35V, Vault:FP-C3216-160-0_2-IPC_B
- removed C1100: GMK107BJ104KAHT, Vault:FP-0603-L_1_6_0_1-W_0_8_0-IPC_B
- removed C1101, C1102: 1uF, Vault:FP-CGA3E-0_3-0_1-MFG
- removed C1103: Capacitor 22µF +/-40% 16V 0805, Vault:CAPC0805(2012)145_L
- removed C900: GRM188R71H472KA01D, Vault:CAPC1608X90X35ML10T15
- removed C901, C902, C903: GRM188R71H104KA93D, Vault:CAPC1608X90X35ML10T15
- removed C904, C905: GRM1885C1H220JA01D, Vault:CAPC1608X90X35ML10T15
- removed D100, D101, D102: 28mm 7-Segment, AltiumLib_MILUTIN.PcbLib:GS8011AR-G
- removed D1001, D1021: MMBZ5231BLT1G, Vault:ONSC-SOT-23-3-318-08_V
- removed D110: 19mm 14-Segment, Alphanummerical, AltiumLib_MILUTIN.PcbLib:GS4011AG-G
- removed D1100: TPD2E1B06DRLR, Vault:FP-DRL0006A-MFG
- removed D1101, D1102, D1103, D1104: SBR80520LT1G, Vault:FP-425-04-MFG
- removed D510, D511, D512, D513, D514, D515, D520, D521, D522, D523: 10mm 7-Segment, AltiumLib_MILUTIN.PcbLib:GS2011AG-G
- removed D900: ESDONCAN1LT3G, Vault:FP-318-MFG
- removed J800, J801: CTB9302/9, AltiumLib_MILUTIN.PcbLib:CTB9302-9
- removed J900: CTB9302/2, AltiumLib_MILUTIN.PcbLib:CTB9302-2
- removed L1001, L1021: IHLP5050CEER1R5M01, AltiumLib_MILUTIN.PcbLib:IHLP5050CEER1R5M01
- removed L900: ACT45B-101-2P-TL003, Vault:FP-ACT45B-MFG
- removed M* (x6): Passermarke, C__ProgramData_Altium_Altium Designer {C630E62D-A531-4285-830B-D4191BD85BC5}_VaultsFileCache_56503fbfafdd0bb88c36dd0b78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
- removed P001: 3P-SMD/THT, AltiumLib_MILUTIN.PcbLib:3P-SMD/THT
- removed P1100: TYPEC-300D-BCP16H100, Vault:TYPEC-300D-BCP16H100-Footprint-1
- removed P1101, P1103: 5-146130-2, Vault:TECO-5-146130-2_V
- removed P1102: M20-8770442R, AltiumLib_MILUTIN.PcbLib:HARWIN_M20-8770442R
- removed P1104: HTSS-105-01-L-DV, Vault:SMTC-HTSS-105-01-X-DV
- removed PTH1, PTH2, PTH3, PTH4, PTH5, PTH6, PTH7, PTH8: PTH-M4D7X7, C__ProgramData_Altium_Altium Designer {C630E62D-A531-4285-830B-D4191BD85BC5}_VaultsFileCache_23ed18ddfbb220747f810c4c6e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
- removed Q1103, Q1104: DTC123JET1G, Vault:ONSC-SC-75-3-463-01_V
- removed R000, R001, R002, R003, R004, R005, R006, R007, R840, R841, R842, R843, R844, R845: RC0603JR-070RL, Vault:RESC1608X55X25ML10T15
- removed R100, R101, R102, R110, R111, R510, R511, R512, R513, R514, R515, R520, R521, R522, R523: 680Ω, Vault:FP-CRCW0603-e3-IPC_A
- removed R1001, R1002, R1021, R1022: 20k/1%, Vault:FP-RC0603-0_55-IPC_C
- removed R1003, R1023: RC0603FR-07100KL, Vault:FP-RC0603-0_55-MFG
- removed R1004: 91k, Vault:RESC1609X50X30NL10T20
- removed R1005, R1025: 20K/1%, Vault:FP-RC0603-0_55-IPC_C
- removed R1024: 150K, Vault:RESC1608X55X30NL15T15
- removed R1100, R1103, R1104, R600: 1kΩ, Vault:FP-CRCW0603-e3-MFG
- removed R1101, R1102: CRCW06035K10FKEA, Vault:FP-CRCW0603-e3-IPC_C
- removed R800, R801, R802, R803, R810, R811, R812, R813, R820, R821, R822, R823, R830, R831, R832, R833: AC0603FR-071KL, Vault:FP-AC0603-IPC_B
- removed R900, R901, R903: CRCW06034K70FKEA, Vault:FP-CRCW0603-e3-IPC_A
- removed R902: CRCW0603120RFKEA, Vault:FP-CRCW0603-e3-MFG
- removed S1100, S1101, S1103, S1104, S600: , Vault:FP-PTS645SM43SMTR92LFS-MFG
- removed U100, U101, U102, U110, U111, U510, U511, U512, U513, U514, U515, U520, U521, U522, U523: TLC59108IPWR, Vault:PW0020A_M
- removed U1000, U1020: TPS51385, AltiumLib_MILUTIN.PcbLib:TPS51386
- removed U1100: ESP32WroomS3, Vault:ESP32WroomS3
- removed U300, U301, U302, U303, U304, U305, U306, U307, U310, U311, U312, U313, U314, U320, U321, U322, U323, U400, U401, U402, U403, U404, U405, U406, U407, U410, U411, U412, U413, U414, U420, U421, U422, U423, U424, U700, U701, U702, U703, U704, U705, U706, U707, U708, U709, U710, U711, U712: WS2812B-4020_2, AltiumLib_MILUTIN.PcbLib:LED_WS2812B-4020
- removed U800, U810, U820, U830: CD40109BQNSR, Vault:FP-NS0016A-IPC_C
- removed U840: MCP23017-E/SS, Vault:SSOP-SS28_N
- removed U900: MCP2562FDT-E/SN, Vault:FP-C04-057-SN-MFG
- removed U901: MCP2515-I/SO, Vault:FP-C04-051-MFG
- removed Y900: ABLS-16.000MHZ-K4T, Vault:FP-ABLS-MFG
- added U224: WS2812B-4020_2, LED_SMD:LED_WS2812B-2020_PLCC4_2.0x2.0mm, F.Cu at (187.0, -80.0)
- added U225: WS2812B-4020_2, LED_SMD:LED_WS2812B-2020_PLCC4_2.0x2.0mm, F.Cu at (190.5, -80.0)
- added U226: WS2812B-4020_2, LED_SMD:LED_WS2812B-2020_PLCC4_2.0x2.0mm, F.Cu at (194.0, -80.0)
- added U227: WS2812B-4020_2, LED_SMD:LED_WS2812B-2020_PLCC4_2.0x2.0mm, F.Cu at (197.5, -80.0)
- added U228: WS2812B-4020_2, LED_SMD:LED_WS2812B-2020_PLCC4_2.0x2.0mm, F.Cu at (201.0, -80.0)
- added U229: WS2812B-4020_2, LED_SMD:LED_WS2812B-2020_PLCC4_2.0x2.0mm, F.Cu at (204.5, -80.0)
- added U230: WS2812B-4020_2, LED_SMD:LED_WS2812B-2020_PLCC4_2.0x2.0mm, F.Cu at (208.0, -79.9)
- added U231: WS2812B-4020_2, LED_SMD:LED_WS2812B-2020_PLCC4_2.0x2.0mm, F.Cu at (211.5, -79.9)
- added U232: WS2812B-4020_2, LED_SMD:LED_WS2812B-2020_PLCC4_2.0x2.0mm, F.Cu at (215.0, -79.9)
- added U233: WS2812B-4020_2, LED_SMD:LED_WS2812B-2020_PLCC4_2.0x2.0mm, F.Cu at (218.5, -79.9)
- added U234: WS2812B-4020_2, LED_SMD:LED_WS2812B-2020_PLCC4_2.0x2.0mm, F.Cu at (222.0, -79.9)
- added U235: WS2812B-4020_2, LED_SMD:LED_WS2812B-2020_PLCC4_2.0x2.0mm, F.Cu at (225.5, -79.9)
- added U236: WS2812B-4020_2, LED_SMD:LED_WS2812B-2020_PLCC4_2.0x2.0mm, F.Cu at (229.0, -80.0)
- added U237: WS2812B-4020_2, LED_SMD:LED_WS2812B-2020_PLCC4_2.0x2.0mm, F.Cu at (232.5, -80.0)
- added U238: WS2812B-4020_2, LED_SMD:LED_WS2812B-2020_PLCC4_2.0x2.0mm, F.Cu at (236.0, -80.0)
- added U239: WS2812B-4020_2, LED_SMD:LED_WS2812B-2020_PLCC4_2.0x2.0mm, F.Cu at (239.5, -80.0)
- added U240: WS2812B-4020_2, LED_SMD:LED_WS2812B-2020_PLCC4_2.0x2.0mm, F.Cu at (243.0, -80.0)
- added U241: WS2812B-4020_2, LED_SMD:LED_WS2812B-2020_PLCC4_2.0x2.0mm, F.Cu at (246.5, -80.0)
- U204, U205, U206, U207, U208, U209, U210, U211, U212, U213, U214, U215, U216, U217, U218, U219, U220, U221, U222, U223: footprint AltiumLib_MILUTIN.PcbLib:LED_WS2812B-4020 -> LED_SMD:LED_WS2812B-2020_PLCC4_2.0x2.0mm
- moved U223 164.4 mm to (183.5, -80.0), turned to 180 degrees
- moved U222 163.7 mm to (180.0, -80.0), turned to 180 degrees
- moved U221 163.0 mm to (176.5, -80.0), turned to 180 degrees
- moved U220 162.4 mm to (173.0, -80.0), turned to 180 degrees
- moved U219 158.0 mm to (171.8, -76.7), turned to -20 degrees
- moved U218 153.7 mm to (170.6, -73.4), turned to -20 degrees
- moved U217 149.6 mm to (169.4, -70.2), turned to -20 degrees
- moved U204 149.4 mm to (153.8, -27.4), turned to -20 degrees
- moved U205 147.0 mm to (155.0, -30.7), turned to -20 degrees
- moved U216 145.5 mm to (168.2, -66.9), turned to -20 degrees
- moved U206 144.7 mm to (156.2, -34.0), turned to -20 degrees
- moved U207 142.3 mm to (157.4, -37.3), turned to -20 degrees
- moved U215 141.6 mm to (167.0, -63.6), turned to -20 degrees
- moved U208 140.0 mm to (158.6, -40.6), turned to -20 degrees
- moved U214 137.8 mm to (165.8, -60.3), turned to -20 degrees
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Connections:
- U204 pad 1: NetU204_1 -> Net-(U204-DOUT)
- U204 pad 2: 5V -> GND
- U204 pad 3: NetU204_3 -> /Designator/NeoPixelData
- U204 pad 4: GND -> 5V
- U205 pad 1: NetU204_3 -> Net-(U205-DOUT)
- U205 pad 2: 5V -> GND
- U205 pad 3: NetU205_3 -> Net-(U204-DOUT)
- U205 pad 4: GND -> 5V
- U206 pad 1: NetU205_3 -> Net-(U206-DOUT)
- U206 pad 2: 5V -> GND
- U206 pad 3: NetU206_3 -> Net-(U205-DOUT)
- U206 pad 4: GND -> 5V
- U207 pad 1: NetU206_3 -> Net-(U207-DOUT)
- U207 pad 2: 5V -> GND
- U207 pad 3: NetU207_3 -> Net-(U206-DOUT)
- U207 pad 4: GND -> 5V
- U208 pad 1: NetU207_3 -> Net-(U208-DOUT)
- U208 pad 2: 5V -> GND
- U208 pad 3: NetU208_3 -> Net-(U207-DOUT)
- U208 pad 4: GND -> 5V
- U209 pad 1: NetU208_3 -> Net-(U209-DOUT)
- U209 pad 2: 5V -> GND
- U209 pad 3: NetU209_3 -> Net-(U208-DOUT)
- U209 pad 4: GND -> 5V
- U210 pad 1: NetU209_3 -> Net-(U210-DOUT)
- U210 pad 2: 5V -> GND
- U210 pad 3: NetU210_3 -> Net-(U209-DOUT)
- U210 pad 4: GND -> 5V
- U211 pad 1: NetU210_3 -> Net-(U211-DOUT)
- U211 pad 2: 5V -> GND
- U211 pad 3: NetU211_3 -> Net-(U210-DOUT)
- U211 pad 4: GND -> 5V
- U212 pad 1: NetU211_3 -> Net-(U212-DOUT)
- U212 pad 2: 5V -> GND
- U212 pad 3: NetU212_3 -> Net-(U211-DOUT)
- U212 pad 4: GND -> 5V
- U213 pad 1: NetU212_3 -> Net-(U213-DOUT)
- U213 pad 2: 5V -> GND
- U213 pad 3: NetU213_3 -> Net-(U212-DOUT)
- U213 pad 4: GND -> 5V
- U214 pad 1: NetU213_3 -> Net-(U214-DOUT)
- U214 pad 2: 5V -> GND
- U214 pad 3: NetU214_3 -> Net-(U213-DOUT)
- U214 pad 4: GND -> 5V
- U215 pad 1: NetU214_3 -> Net-(U215-DOUT)
- U215 pad 2: 5V -> GND
- U215 pad 3: NetU215_3 -> Net-(U214-DOUT)
- U215 pad 4: GND -> 5V
- U216 pad 1: NetU215_3 -> Net-(U216-DOUT)
- U216 pad 2: 5V -> GND
- U216 pad 3: NetU216_3 -> Net-(U215-DOUT)
- U216 pad 4: GND -> 5V
- U217 pad 1: NetU216_3 -> Net-(U217-DOUT)
- U217 pad 2: 5V -> GND
- U217 pad 3: NetU217_3 -> Net-(U216-DOUT)
- U217 pad 4: GND -> 5V
- U218 pad 1: NetU217_3 -> Net-(U218-DOUT)
- U218 pad 2: 5V -> GND
- U218 pad 3: NetU218_3 -> Net-(U217-DOUT)
- U218 pad 4: GND -> 5V
- U219 pad 1: NetU218_3 -> Net-(U219-DOUT)
- U219 pad 2: 5V -> GND
- U219 pad 3: NetU219_3 -> Net-(U218-DOUT)
- U219 pad 4: GND -> 5V
- U220 pad 1: NetU219_3 -> Net-(U220-DOUT)
- U220 pad 2: 5V -> GND
- U220 pad 3: NetU220_3 -> Net-(U219-DOUT)
- U220 pad 4: GND -> 5V
- U221 pad 1: NetU220_3 -> Net-(U221-DOUT)
- U221 pad 2: 5V -> GND
- U221 pad 3: NetU221_3 -> Net-(U220-DOUT)
- U221 pad 4: GND -> 5V
- U222 pad 1: NetU221_3 -> Net-(U222-DOUT)
- U222 pad 2: 5V -> GND
- U222 pad 3: NetU222_3 -> Net-(U221-DOUT)
- U222 pad 4: GND -> 5V
- U223 pad 1: NetU222_3 -> Net-(U223-DOUT)
- U223 pad 2: 5V -> GND
- U223 pad 3: NetU223_3 -> Net-(U222-DOUT)
- U223 pad 4: GND -> 5V
Routing:
- net (no net): track 0.00 -> 5732.6 mm, vias 33 -> 371
- net SDA: track 329.4 -> 0.00 mm, vias 20 -> 0
- net SCL: track 329.3 -> 0.00 mm, vias 20 -> 0
- net ~{DIG-RST}: track 301.5 -> 0.00 mm, vias 18 -> 0
- net KL30: track 186.5 -> 0.00 mm, vias 16 -> 0
- net NetR600_2: track 124.1 -> 0.00 mm, vias 4 -> 0
- net KL30i: track 123.3 -> 0.00 mm, vias 4 -> 0
- net EN: track 114.9 -> 0.00 mm, vias 6 -> 0
- net NetU223_3: track 101.0 -> 0.00 mm, vias 4 -> 0
- net VBUS: track 88.7 -> 0.00 mm, vias 6 -> 0
- net 5V: track 403.0 -> 323.1 mm, vias 116 -> 105
- net NetS1101_3: track 76.4 -> 0.00 mm, vias 4 -> 0
- net NetP001_2: track 63.6 -> 0.00 mm, vias 2 -> 0
- net RX: track 59.1 -> 0.00 mm, vias 3 -> 0
- net TX: track 56.2 -> 0.00 mm, vias 4 -> 0
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- added copper zone on B.Cu, net (none)
- added copper zone on In2.Cu, net (none)
- removed copper zone on B.Cu, net 3V3
- removed copper zone on In2.Cu, net 3V3
- removed copper zone on B.Cu, net KL30
- removed copper zone on B.Cu, net KL30i
- removed copper zone on B.Cu, net KL31
- removed copper zone on B.Cu, net NetC1006_1
- removed copper zone on B.Cu, net NetC1026_1

Commit message: current version of lada speedometer in kicad
Parts:
- added C900: C 1uF, Capacitor_SMD:C_0603_1608Metric, F.Cu at (45.6, 60.1)
- added C901: C 1uF, Capacitor_SMD:C_0603_1608Metric, F.Cu at (45.6, 62.6)
- added C902: C 1uF, Capacitor_SMD:C_0603_1608Metric, F.Cu at (45.6, 65.2)
- added C903: 22pF, Capacitor_SMD:C_0603_1608Metric, F.Cu at (45.6, 67.7)
- added C904: 22pF, Capacitor_SMD:C_0603_1608Metric, F.Cu at (45.6, 70.2)
- added FID1: Fiducial, Fiducial:Fiducial_0.5mm_Mask1mm, F.Cu at (-22.9, 49.5)
- added FID2: Fiducial, Fiducial:Fiducial_0.5mm_Mask1mm, F.Cu at (-22.9, 52.0)
- added FID3: Fiducial, Fiducial:Fiducial_0.5mm_Mask1mm, F.Cu at (-20.3, 49.5)
- added FID4: Fiducial, Fiducial:Fiducial_0.5mm_Mask1mm, F.Cu at (-20.3, 52.0)
- added FID5: Fiducial, Fiducial:Fiducial_0.5mm_Mask1mm, F.Cu at (-17.8, 49.5)
- added FID6: Fiducial, Fiducial:Fiducial_0.5mm_Mask1mm, F.Cu at (-17.8, 52.0)
- added H1: MountingHole, MountingHole:MountingHole_4.3mm_M4_ISO7380, F.Cu at (5.00, -98.7)
- added H2: MountingHole, MountingHole:MountingHole_4.3mm_M4_ISO7380, F.Cu at (5.00, -25.0)
- added H3: MountingHole, MountingHole:MountingHole_4.3mm_M4_ISO7380, F.Cu at (95.0, -98.7)
- added H4: MountingHole, MountingHole:MountingHole_4.3mm_M4_ISO7380, F.Cu at (95.0, -25.0)
- added H5: MountingHole, MountingHole:MountingHole_4.3mm_M4_ISO7380, F.Cu at (214.2, -98.7)
- added H6: MountingHole, MountingHole:MountingHole_4.3mm_M4_ISO7380, F.Cu at (214.2, -25.0)
- added H7: MountingHole, MountingHole:MountingHole_4.3mm_M4_ISO7380, F.Cu at (304.2, -98.7)
- added H8: MountingHole, MountingHole:MountingHole_4.3mm_M4_ISO7380, F.Cu at (304.2, -25.0)
- added J1: Conn_01x03_Pin, Connector_PinHeader_2.54mm:PinHeader_1x03_P2.54mm_Horizontal, F.Cu at (19.0, -97.1)
- added J800: 776228-1, Connector_TE-Connectivity:TE_776228-1, B.Cu at (115.0, 32.0)
- added R609: R 1k, Resistor_SMD:R_0201_0603Metric, F.Cu at (75.0, 59.8)
- added R610: R 1k, Resistor_SMD:R_0201_0603Metric, F.Cu at (75.0, 61.5)
- added R8: R 4k7, Resistor_SMD:R_0603_1608Metric, F.Cu at (45.6, 72.7)
- added R9: 1k, Resistor_SMD:R_0603_1608Metric, F.Cu at (15.3, 15.4)
- added R900: R 120, Resistor_SMD:R_0603_1608Metric, F.Cu at (45.6, 75.2)
- added S600: SW_Omron_B3FS, Button_Switch_SMD:SW_SPST_Omron_B3FS-100xP, F.Cu at (25.1, -39.6)
- added S601: SW_Omron_B3FS, Button_Switch_SMD:SW_SPST_Omron_B3FS-100xP, F.Cu at (68.2, 62.8)
- added S602: SW_Omron_B3FS, Button_Switch_SMD:SW_SPST_Omron_B3FS-100xP, F.Cu at (68.2, 70.7)
- added TP1: TestPoint_Probe, TestPoint:TestPoint_Pad_2.0x2.0mm, F.Cu at (16.0, 86.0)
- added TP2: TestPoint_Probe, TestPoint:TestPoint_Pad_2.0x2.0mm, F.Cu at (16.0, 90.0)
- added U1: MCP23017_SS, Package_SO:SSOP-28_5.3x10.2mm_P0.65mm, F.Cu at (3.00, 91.0)
- added U100: TLC59108IPWR, Package_SO:TSSOP-20_4.4x6.5mm_P0.65mm, B.Cu at (223.1, -52.2)
- added U101: TLC59108IPWR, Package_SO:TSSOP-20_4.4x6.5mm_P0.65mm, B.Cu at (206.1, -52.2)
- added U102: TLC59108IPWR, Package_SO:TSSOP-20_4.4x6.5mm_P0.65mm, B.Cu at (189.1, -52.2)
- added U110: TLC59108IPWR, Package_SO:TSSOP-20_4.4x6.5mm_P0.65mm, B.Cu at (154.5, -69.5)
- added U111: TLC59108IPWR, Package_SO:TSSOP-20_4.4x6.5mm_P0.65mm, B.Cu at (154.5, -77.5)
- added U2: TLC59108xPW, Package_SO:TSSOP-20_4.4x6.5mm_P0.65mm, F.Cu at (332.0, 23.5)
- added U3: 4010, Package_DIP:DIP-16_W7.62mm_LongPads, F.Cu at (-0.76, 55.2)
- added U301: WS2812B-4020_2, LED_SMD:LED_WS2812B-2020_PLCC4_2.0x2.0mm, F.Cu at (299.2, -32.2)
- added U302: WS2812B-4020_2, LED_SMD:LED_WS2812B-2020_PLCC4_2.0x2.0mm, F.Cu at (299.2, -35.8)
- added U303: WS2812B-4020_2, LED_SMD:LED_WS2812B-2020_PLCC4_2.0x2.0mm, F.Cu at (299.2, -39.2)
- added U304: WS2812B-4020_2, LED_SMD:LED_WS2812B-2020_PLCC4_2.0x2.0mm, F.Cu at (299.2, -42.8)
- added U305: WS2812B-4020_2, LED_SMD:LED_WS2812B-2020_PLCC4_2.0x2.0mm, F.Cu at (299.2, -46.2)
- added U306: WS2812B-4020_2, LED_SMD:LED_WS2812B-2020_PLCC4_2.0x2.0mm, F.Cu at (299.2, -49.8)
- added U307: WS2812B-4020_2, LED_SMD:LED_WS2812B-2020_PLCC4_2.0x2.0mm, F.Cu at (299.2, -53.2)
- added U308: WS2812B-4020_2, LED_SMD:LED_WS2812B-2020_PLCC4_2.0x2.0mm, F.Cu at (299.1, -56.8)
- added U309: WS2812B-4020_2, LED_SMD:LED_WS2812B-2020_PLCC4_2.0x2.0mm, F.Cu at (299.1, -60.2)
- added U310: WS2812B-4020_2, LED_SMD:LED_WS2812B-2020_PLCC4_2.0x2.0mm, F.Cu at (299.2, -63.8)
- added U311: WS2812B-4020_2, LED_SMD:LED_WS2812B-2020_PLCC4_2.0x2.0mm, F.Cu at (299.2, -67.2)
- added U312: WS2812B-4020_2, LED_SMD:LED_WS2812B-2020_PLCC4_2.0x2.0mm, F.Cu at (299.2, -70.8)
- added U313: WS2812B-4020_2, LED_SMD:LED_WS2812B-2020_PLCC4_2.0x2.0mm, F.Cu at (299.2, -74.2)
- added U314: WS2812B-4020_2, LED_SMD:LED_WS2812B-2020_PLCC4_2.0x2.0mm, F.Cu at (299.2, -77.8)
- added U315: WS2812B-4020_2, LED_SMD:LED_WS2812B-2020_PLCC4_2.0x2.0mm, F.Cu at (299.2, -81.2)
- added U316: WS2812B-4020_2, LED_SMD:LED_WS2812B-2020_PLCC4_2.0x2.0mm, F.Cu at (299.2, -84.8)
- added U317: WS2812B-4020_2, LED_SMD:LED_WS2812B-2020_PLCC4_2.0x2.0mm, F.Cu at (294.2, -86.5)
- added U318: WS2812B-4020_2, LED_SMD:LED_WS2812B-2020_PLCC4_2.0x2.0mm, F.Cu at (289.2, -86.5)
- added U319: WS2812B-4020_2, LED_SMD:LED_WS2812B-2020_PLCC4_2.0x2.0mm, F.Cu at (294.2, -72.5)
- added U320: WS2812B-4020_2, LED_SMD:LED_WS2812B-2020_PLCC4_2.0x2.0mm, F.Cu at (289.2, -72.5)
- added U321: WS2812B-4020_2, LED_SMD:LED_WS2812B-2020_PLCC4_2.0x2.0mm, F.Cu at (294.2, -58.5)
- added U322: WS2812B-4020_2, LED_SMD:LED_WS2812B-2020_PLCC4_2.0x2.0mm, F.Cu at (289.2, -58.5)
- added U323: WS2812B-4020_2, LED_SMD:LED_WS2812B-2020_PLCC4_2.0x2.0mm, F.Cu at (294.2, -44.5)
- added U324: WS2812B-4020_2, LED_SMD:LED_WS2812B-2020_PLCC4_2.0x2.0mm, F.Cu at (289.2, -44.5)
- added U325: WS2812B-4020_2, LED_SMD:LED_WS2812B-2020_PLCC4_2.0x2.0mm, F.Cu at (294.2, -30.5)
- added U326: WS2812B-4020_2, LED_SMD:LED_WS2812B-2020_PLCC4_2.0x2.0mm, F.Cu at (289.2, -30.5)
- added U4: 4010, Package_DIP:DIP-16_W7.62mm_LongPads, F.Cu at (10.8, 55.2)
- added U401: WS2812B-4020_2, LED_SMD:LED_WS2812B-2020_PLCC4_2.0x2.0mm, F.Cu at (10.0, -32.2)
- added U402: WS2812B-4020_2, LED_SMD:LED_WS2812B-2020_PLCC4_2.0x2.0mm, F.Cu at (10.0, -35.8)
- added U403: WS2812B-4020_2, LED_SMD:LED_WS2812B-2020_PLCC4_2.0x2.0mm, F.Cu at (10.0, -39.2)
- added U404: WS2812B-4020_2, LED_SMD:LED_WS2812B-2020_PLCC4_2.0x2.0mm, F.Cu at (10.0, -42.8)
- added U405: WS2812B-4020_2, LED_SMD:LED_WS2812B-2020_PLCC4_2.0x2.0mm, F.Cu at (10.0, -46.2)
- added U406: WS2812B-4020_2, LED_SMD:LED_WS2812B-2020_PLCC4_2.0x2.0mm, F.Cu at (10.0, -49.8)
- added U407: WS2812B-4020_2, LED_SMD:LED_WS2812B-2020_PLCC4_2.0x2.0mm, F.Cu at (10.0, -53.2)
- added U408: WS2812B-4020_2, LED_SMD:LED_WS2812B-2020_PLCC4_2.0x2.0mm, F.Cu at (10.0, -56.8)
- added U409: WS2812B-4020_2, LED_SMD:LED_WS2812B-2020_PLCC4_2.0x2.0mm, F.Cu at (10.0, -60.2)
- added U410: WS2812B-4020_2, LED_SMD:LED_WS2812B-2020_PLCC4_2.0x2.0mm, F.Cu at (10.0, -63.8)
- added U411: WS2812B-4020_2, LED_SMD:LED_WS2812B-2020_PLCC4_2.0x2.0mm, F.Cu at (10.0, -67.2)
- added U412: WS2812B-4020_2, LED_SMD:LED_WS2812B-2020_PLCC4_2.0x2.0mm, F.Cu at (10.0, -70.8)
- added U413: WS2812B-4020_2, LED_SMD:LED_WS2812B-2020_PLCC4_2.0x2.0mm, F.Cu at (10.0, -74.2)
- added U414: WS2812B-4020_2, LED_SMD:LED_WS2812B-2020_PLCC4_2.0x2.0mm, F.Cu at (10.0, -77.8)
- added U415: WS2812B-4020_2, LED_SMD:LED_WS2812B-2020_PLCC4_2.0x2.0mm, F.Cu at (10.0, -81.2)
- added U416: WS2812B-4020_2, LED_SMD:LED_WS2812B-2020_PLCC4_2.0x2.0mm, F.Cu at (10.0, -84.8)
- added U417: WS2812B-4020_2, LED_SMD:LED_WS2812B-2020_PLCC4_2.0x2.0mm, F.Cu at (15.0, -86.5)
- added U418: WS2812B-4020_2, LED_SMD:LED_WS2812B-2020_PLCC4_2.0x2.0mm, F.Cu at (20.0, -86.5)
- added U419: WS2812B-4020_2, LED_SMD:LED_WS2812B-2020_PLCC4_2.0x2.0mm, F.Cu at (15.0, -72.5)
- added U420: WS2812B-4020_2, LED_SMD:LED_WS2812B-2020_PLCC4_2.0x2.0mm, F.Cu at (20.0, -72.5)
- added U421: WS2812B-4020_2, LED_SMD:LED_WS2812B-2020_PLCC4_2.0x2.0mm, F.Cu at (15.0, -58.5)
- added U422: WS2812B-4020_2, LED_SMD:LED_WS2812B-2020_PLCC4_2.0x2.0mm, F.Cu at (20.0, -58.5)
- added U423: WS2812B-4020_2, LED_SMD:LED_WS2812B-2020_PLCC4_2.0x2.0mm, F.Cu at (15.0, -44.5)
- added U424: WS2812B-4020_2, LED_SMD:LED_WS2812B-2020_PLCC4_2.0x2.0mm, F.Cu at (20.0, -44.5)
- added U425: WS2812B-4020_2, LED_SMD:LED_WS2812B-2020_PLCC4_2.0x2.0mm, F.Cu at (15.0, -30.5)
- added U426: WS2812B-4020_2, LED_SMD:LED_WS2812B-2020_PLCC4_2.0x2.0mm, F.Cu at (20.0, -30.5)
- added U5: 4010, Package_DIP:DIP-16_W7.62mm_LongPads, F.Cu at (22.4, 55.2)
- added U601: ESP32-S3-WROOM-1(N8R2), RF_Module:ESP32-S3-WROOM-2, F.Cu at (131.0, 85.7)
- added U603: CP2102N-A02-GQFN28R, Package_DFN_QFN:VQFN-28-1EP_5x5mm_P0.5mm_EP3.25x3.25mm, F.Cu at (94.0, 92.5)
- added U700: WS2812B-4020_2, LED_SMD:LED_WS2812B-2020_PLCC4_2.0x2.0mm, F.Cu at (299.6, -8.00)
- added U701: WS2812B-4020_2, LED_SMD:LED_WS2812B-2020_PLCC4_2.0x2.0mm, F.Cu at (277.3, -8.00)
- added U702: WS2812B-4020_2, LED_SMD:LED_WS2812B-2020_PLCC4_2.0x2.0mm, F.Cu at (255.0, -8.00)
- added U703: WS2812B-4020_2, LED_SMD:LED_WS2812B-2020_PLCC4_2.0x2.0mm, F.Cu at (232.7, -8.00)
- added U704: WS2812B-4020_2, LED_SMD:LED_WS2812B-2020_PLCC4_2.0x2.0mm, F.Cu at (210.4, -8.00)
- added U705: WS2812B-4020_2, LED_SMD:LED_WS2812B-2020_PLCC4_2.0x2.0mm, F.Cu at (188.1, -8.00)
- added U706: WS2812B-4020_2, LED_SMD:LED_WS2812B-2020_PLCC4_2.0x2.0mm, F.Cu at (154.6, -8.00)
- added U707: WS2812B-4020_2, LED_SMD:LED_WS2812B-2020_PLCC4_2.0x2.0mm, F.Cu at (121.1, -8.00)
- added U708: WS2812B-4020_2, LED_SMD:LED_WS2812B-2020_PLCC4_2.0x2.0mm, F.Cu at (98.8, -8.00)
- added U709: WS2812B-4020_2, LED_SMD:LED_WS2812B-2020_PLCC4_2.0x2.0mm, F.Cu at (76.5, -8.00)
- added U710: WS2812B-4020_2, LED_SMD:LED_WS2812B-2020_PLCC4_2.0x2.0mm, F.Cu at (54.2, -8.00)
- added U711: WS2812B-4020_2, LED_SMD:LED_WS2812B-2020_PLCC4_2.0x2.0mm, F.Cu at (31.9, -8.00)
- added U712: WS2812B-4020_2, LED_SMD:LED_WS2812B-2020_PLCC4_2.0x2.0mm, F.Cu at (9.64, -8.00)
- added U900: MCP2562-H-SN, Package_SO:SOIC-8_3.9x4.9mm_P1.27mm, F.Cu at (51.9, 75.5)
- added U902: MCP2515-xSO, Package_SO:SOIC-18W_7.5x11.6mm_P1.27mm, F.Cu at (54.1, 65.5)
Connections:
- U204 pad 3: /Designator/NeoPixelData -> /Torq/TorqIn
- U241 pad 1: /Designator/SocIn -> /SOC/SocIn
Routing:
- net (no net): track 5732.6 -> 2234.5 mm, vias 371 -> 207
- net Net-(U101-~{OUT0}): track 0.00 -> 145.4 mm, vias 0 -> 8
- net GND: track 398.0 -> 278.8 mm, vias 188 -> 118
- net 5V: track 323.1 -> 282.0 mm, vias 105 -> 75
- net /Distance/~{DIG-RST}: track 0.00 -> 25.9 mm, vias 0 -> 3
- net /Distance/SDA: track 0.00 -> 24.8 mm, vias 0 -> 3
- net Net-(U102-~{OUT7}): track 0.00 -> 21.0 mm, vias 0 -> 1
- net Net-(U101-~{OUT7}): track 0.00 -> 19.4 mm, vias 0 -> 1
- net Net-(U100-~{OUT7}): track 0.00 -> 19.4 mm, vias 0 -> 1
- net Net-(U102-~{OUT3}): track 0.00 -> 16.5 mm, vias 0 -> 2
- net Net-(U102-~{OUT5}): track 0.00 -> 15.9 mm, vias 0 -> 1
- net Net-(U101-~{OUT2}): track 0.00 -> 15.8 mm, vias 0 -> 1
- net Net-(U100-~{OUT2}): track 0.00 -> 15.8 mm, vias 0 -> 1
- net Net-(U102-~{OUT2}): track 0.00 -> 15.5 mm, vias 0 -> 1
- net Net-(U101-~{OUT3}): track 0.00 -> 15.0 mm, vias 0 -> 1
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Other:
- board text removed: "I2C"
- board text removed: "JTAG"
- board text removed: "L CAN H"
- board text removed: "SERIAL"

Commit message: Speedometer DRC mostly passed
Parts:
- removed U2: TLC59108xPW, Package_SO:TSSOP-20_4.4x6.5mm_P0.65mm
- removed U204: WS2812B-4020_2, LED_SMD:LED_WS2812B-2020_PLCC4_2.0x2.0mm
- added C1001: 10uF, Capacitor_SMD:C_0805_2012Metric, B.Cu at (138.0, -42.0)
- added C1002: 10uF, Capacitor_SMD:C_0805_2012Metric, B.Cu at (138.0, -39.0)
- added C1003: 100nF, Capacitor_SMD:C_0805_2012Metric, B.Cu at (129.5, -43.0)
- added C1004: 22uF, Capacitor_SMD:C_0805_2012Metric, B.Cu at (135.5, -58.0)
- added C1005: 22uF, Capacitor_SMD:C_0805_2012Metric, B.Cu at (132.5, -58.0)
- added C1011: 10uF, Capacitor_SMD:C_0805_2012Metric, B.Cu at (118.0, -39.0)
- added C1012: 10uF, Capacitor_SMD:C_0805_2012Metric, B.Cu at (118.0, -42.0)
- added C1013: 100nF, Capacitor_SMD:C_0805_2012Metric, B.Cu at (109.5, -43.0)
- added C1014: 22uF, Capacitor_SMD:C_0805_2012Metric, B.Cu at (115.5, -57.5)
- added C1015: 22uF, Capacitor_SMD:C_0805_2012Metric, B.Cu at (112.5, -57.5)
- added C601: 1uF, Capacitor_SMD:C_0805_2012Metric, B.Cu at (139.5, -94.5)
- added C602: 22uF, Capacitor_SMD:C_0805_2012Metric, B.Cu at (136.5, -95.5)
- added C603: 100nF, Capacitor_SMD:C_0201_0603Metric, B.Cu at (135.0, -95.5)
- added C605: 100nF, Resistor_SMD:R_0603_1608Metric, B.Cu at (90.0, -85.0)
- added D100: ~, Display_7Segment:GS8011AR-G, F.Cu at (223.1, -49.5)
- added D101: ~, Display_7Segment:GS8011AR-G, F.Cu at (206.1, -49.5)
- added D102: ~, Display_7Segment:GS8011AR-G, F.Cu at (189.1, -49.5)
- added D110: GS4011AG-G, Display_7Segment:GS4011AG-G, F.Cu at (154.6, -73.0)
- added D510: 10mm 7-Segment, Display_7Segment:GS2011AG-G, F.Cu at (90.3, -49.6)
- added D511: 10mm 7-Segment, Display_7Segment:GS2011AG-G, F.Cu at (83.3, -49.6)
- added D512: 10mm 7-Segment, Display_7Segment:GS2011AG-G, F.Cu at (76.3, -49.6)
- added D513: 10mm 7-Segment, Display_7Segment:GS2011AG-G, F.Cu at (69.3, -49.6)
- added D514: 10mm 7-Segment, Display_7Segment:GS2011AG-G, F.Cu at (62.3, -49.6)
- added D515: 10mm 7-Segment, Display_7Segment:GS2011AG-G, F.Cu at (55.3, -49.6)
- added D520: 10mm 7-Segment, Display_7Segment:GS2011AG-G, F.Cu at (83.3, -29.6)
- added D521: 10mm 7-Segment, Display_7Segment:GS2011AG-G, F.Cu at (76.3, -29.6)
- added D522: 10mm 7-Segment, Display_7Segment:GS2011AG-G, F.Cu at (69.3, -29.6)
- added D523: 10mm 7-Segment, Display_7Segment:GS2011AG-G, F.Cu at (62.3, -29.6)
- added H602: 2x3, Connector_PinHeader_2.54mm:PinHeader_2x03_P2.54mm_Vertical_SMD, B.Cu at (154.5, -92.5)
- added L1001: SRN8040-2R2Y, Inductor_SMD:L_Bourns-SRN8040_8x8.15mm, B.Cu at (134.0, -50.5)
- added L1011: SRN8040-3R3Y, Inductor_SMD:L_Bourns-SRN8040_8x8.15mm, B.Cu at (114.0, -50.3)
- added Q601: DTC123J, Package_TO_SOT_SMD:SOT-23, B.Cu at (136.0, -73.5)
- added Q602: DTC123J, Package_TO_SOT_SMD:SOT-23, B.Cu at (140.5, -73.5)
- added R000: 0, Resistor_SMD:R_0603_1608Metric, B.Cu at (43.0, -80.5)
- added R001: 0, Resistor_SMD:R_0603_1608Metric, B.Cu at (41.5, -80.5)
- added R002: 0, Resistor_SMD:R_0603_1608Metric, B.Cu at (36.5, -80.5)
- added R003: 0, Resistor_SMD:R_0603_1608Metric, B.Cu at (35.0, -80.5)
- added R100: 680, Resistor_SMD:R_0603_1608Metric, B.Cu at (223.2, -57.0)
- added R1001: 33.2k, Resistor_SMD:R_0603_1608Metric, B.Cu at (126.0, -47.5)
- added R1002: 10k, Resistor_SMD:R_0603_1608Metric, B.Cu at (124.0, -47.5)
- added R101: 680, Resistor_SMD:R_0603_1608Metric, B.Cu at (206.2, -57.0)
- added R1011: 56.2k, Resistor_SMD:R_0603_1608Metric, B.Cu at (106.0, -47.5)
- added R1012: 10k, Resistor_SMD:R_0603_1608Metric, B.Cu at (104.0, -47.5)
- added R102: 680, Resistor_SMD:R_0603_1608Metric, B.Cu at (189.0, -57.0)
- added R11: 0R, Resistor_SMD:R_0603_1608Metric, B.Cu at (92.2, -78.8)
- added R110: 680, Resistor_SMD:R_0603_1608Metric, B.Cu at (162.8, -78.9)
- added R111: 680, Resistor_SMD:R_0603_1608Metric, B.Cu at (162.8, -73.0)
- added R12: 0R, Resistor_SMD:R_0603_1608Metric, B.Cu at (93.8, -78.8)
- added R13: 0R, Resistor_SMD:R_0603_1608Metric, B.Cu at (95.2, -78.8)
- added R14: 0R, Resistor_SMD:R_0603_1608Metric, B.Cu at (92.2, -75.2)
- added R15: 0R, Resistor_SMD:R_0603_1608Metric, B.Cu at (93.8, -75.2)
- added R16: 0R, Resistor_SMD:R_0603_1608Metric, B.Cu at (95.2, -75.2)
- added R17: 0R, Resistor_SMD:R_0603_1608Metric, B.Cu at (38.8, -80.5)
- added R18: 0R, Resistor_SMD:R_0603_1608Metric, B.Cu at (44.5, -80.5)
- added R510: 680, Resistor_SMD:R_0603_1608Metric, B.Cu at (94.5, -54.5)
- added R511: 680, Resistor_SMD:R_0603_1608Metric, B.Cu at (90.0, -54.5)
- added R512: 680, Resistor_SMD:R_0603_1608Metric, B.Cu at (78.0, -54.5)
- added R513: 680, Resistor_SMD:R_0603_1608Metric, B.Cu at (73.5, -54.5)
- added R514: 680, Resistor_SMD:R_0603_1608Metric, B.Cu at (61.8, -54.5)
- added R515: 680, Resistor_SMD:R_0603_1608Metric, B.Cu at (57.2, -54.5)
- added R520: 680, Resistor_SMD:R_0603_1608Metric, B.Cu at (86.2, -34.5)
- added R521: 680, Resistor_SMD:R_0603_1608Metric, B.Cu at (81.8, -34.5)
- added R522: 680, Resistor_SMD:R_0603_1608Metric, B.Cu at (69.8, -34.8)
- added R523: 680, Resistor_SMD:R_0603_1608Metric, B.Cu at (65.8, -34.8)
- added R601: 10k, Resistor_SMD:R_0603_1608Metric, B.Cu at (10.0, -74.3)
- added R602: 2.2k, Resistor_SMD:R_0603_1608Metric, B.Cu at (107.5, -93.5)
- added R603: 2.2k, Resistor_SMD:R_0603_1608Metric, B.Cu at (107.5, -95.0)
- added R604: 10k, Resistor_SMD:R_0603_1608Metric, B.Cu at (10.0, -90.1)
- added R605: 10k, Resistor_SMD:R_0603_1608Metric, B.Cu at (100.5, -84.0)
- added R606: 10k, Resistor_SMD:R_0603_1608Metric, B.Cu at (104.5, -84.0)
- added R607: 5.1k, Resistor_SMD:R_0603_1608Metric, F.Cu at (15.0, -51.2)
- added R608: 5.1k, Resistor_SMD:R_0603_1608Metric, F.Cu at (20.8, -53.5)
- added R611: 2.2k, Resistor_SMD:R_0603_1608Metric, B.Cu at (145.5, -76.2)
- added R612: 2.2k, Resistor_SMD:R_0603_1608Metric, B.Cu at (146.5, -81.0)
- added S2: SW_Omron_B3FS, Button_Switch_SMD:SW_SPST_Omron_B3FS-100xP, B.Cu at (17.5, -72.0)
- added S606: SW_Omron_B3FS, Button_Switch_SMD:SW_SPST_Omron_B3FS-100xP, B.Cu at (17.5, -87.9)
- added U1001: TPS563200, Package_TO_SOT_SMD:SOT-23-6, B.Cu at (134.0, -40.5)
- added U1011: TPS563200, Package_TO_SOT_SMD:SOT-23-6, B.Cu at (114.0, -40.5)
- added U510: TLC59108IPWR, Package_SO:TSSOP-20_4.4x6.5mm_P0.65mm, B.Cu at (93.1, -49.6)
- added U511: TLC59108IPWR, Package_SO:TSSOP-20_4.4x6.5mm_P0.65mm, B.Cu at (84.9, -49.6)
- added U512: TLC59108IPWR, Package_SO:TSSOP-20_4.4x6.5mm_P0.65mm, B.Cu at (76.6, -49.6)
- added U513: TLC59108IPWR, Package_SO:TSSOP-20_4.4x6.5mm_P0.65mm, B.Cu at (68.6, -49.6)
- added U514: TLC59108IPWR, Package_SO:TSSOP-20_4.4x6.5mm_P0.65mm, B.Cu at (60.6, -49.6)
- added U515: TLC59108IPWR, Package_SO:TSSOP-20_4.4x6.5mm_P0.65mm, B.Cu at (52.1, -49.6)
- added U520: TLC59108IPWR, Package_SO:TSSOP-20_4.4x6.5mm_P0.65mm, B.Cu at (84.9, -29.6)
- added U521: TLC59108IPWR, Package_SO:TSSOP-20_4.4x6.5mm_P0.65mm, B.Cu at (76.6, -29.6)
- added U522: TLC59108IPWR, Package_SO:TSSOP-20_4.4x6.5mm_P0.65mm, B.Cu at (68.6, -29.6)
- added U523: TLC59108IPWR, Package_SO:TSSOP-20_4.4x6.5mm_P0.65mm, B.Cu at (60.6, -29.6)
- added U602: BC817, Package_TO_SOT_SMD:SOT-23-3, B.Cu at (100.5, -80.0)
- added U604: BC817, Package_TO_SOT_SMD:SOT-23-3, B.Cu at (104.5, -80.0)
- added U605: YTC-TC16S-24, Connector_USB:TYPEC-300D-BCP16H100, F.Cu at (17.5, -51.9)
- added X900: K3A160002010, Crystal:Crystal_SMD_3225-4Pin_3.2x2.5mm, B.Cu at (27.8, -95.0)
- C900, C901, C902, C903, C904, FID2, FID4, FID6, R8, R9, R900, S601, S602, TP1, TP2, U1, U3, U4, U5, U601, U603, U900, U902: moved to B.Cu
- R609, R610: footprint Resistor_SMD:R_0201_0603Metric -> Resistor_SMD:R_0603_1608Metric; moved to B.Cu
- moved FID4 357.1 mm to (306.8, -91.2)
- moved FID3 356.1 mm to (306.8, -91.2)
- moved FID6 329.1 mm to (306.8, -2.50)
- moved FID5 328.7 mm to (306.8, -2.50)
- moved U1 186.5 mm to (84.0, -77.0), turned to -90 degrees
- moved U603 180.0 mm to (95.0, -87.5), turned to 90 degrees
- moved U601 176.6 mm to (124.1, -90.8), turned to 180 degrees
- moved TP2 169.6 mm to (87.0, -64.0)
- moved C904 169.4 mm to (29.8, -98.5), turned to 90 degrees
- moved TP1 163.9 mm to (82.0, -64.0)
- moved R8 159.9 mm to (46.8, -87.2), turned to 90 degrees
- moved C903 159.7 mm to (29.8, -91.2), turned to -90 degrees
- moved U902 158.2 mm to (37.0, -91.8)
- moved U3 157.0 mm to (54.3, -91.8), turned to -90 degrees
- moved C902 151.2 mm to (44.0, -86.0), turned to -90 degrees
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Connections:
- R609 pad 2: Net-(Q601-C) -> /Distance/~{DIG-RST}
- R610 pad 2: Net-(Q602-C) -> /SigIn/~{RESET}
- U100 pad 18: /Distance/SCL -> /Speed/SCL_2
- U100 pad 19: /Distance/SDA -> /Speed/SDA_2
- U100 pad 3: 5V -> GND
- U100 pad 5: 5V -> GND
- U101 pad 18: /Distance/SCL -> /Speed/SCL_2
- U101 pad 19: /Distance/SDA -> /Speed/SDA_2
- U101 pad 3: 5V -> GND
- U101 pad 5: 5V -> GND
- U102 pad 18: /Distance/SCL -> /Speed/SCL_2
- U102 pad 19: /Distance/SDA -> /Speed/SDA_2
- U102 pad 3: GND -> 5V
- U102 pad 4: 5V -> GND
- U102 pad 5: 5V -> GND
- U110 pad 18: /Distance/SCL -> /Speed/SCL_2
- U110 pad 19: /Distance/SDA -> /Speed/SDA_2
- U110 pad 3: GND -> 5V
- U110 pad 4: 5V -> GND
- U110 pad 5: 5V -> GND
- U111 pad 18: /Distance/SCL -> /Speed/SCL_2
- U111 pad 19: /Distance/SDA -> /Speed/SDA_2
- U111 pad 3: 5V -> GND
- U111 pad 5: 5V -> GND
- U205 pad 3: Net-(U204-DOUT) -> /Torq/TorqIn
- U3 pad 16: KL30 -> KL30input
- U4 pad 16: KL30 -> KL30input
- U421 pad 2: GND -> 5V
- U5 pad 11: KL30 -> KL30input
- U5 pad 16: KL30 -> KL30input
- U601 pad 13: unconnected-(U601-IO19-Pad13) -> /Speed/SDA_2
- U601 pad 14: unconnected-(U601-IO20-Pad14) -> /Speed/SCL_2
- U601 pad 2: +3.3V -> 3V3
Routing:
- net (no net): track 2234.5 -> 0.00 mm, vias 207 -> 0
- net /Distance/~{DIG-RST}: track 25.9 -> 374.0 mm, vias 3 -> 21
- net GND: track 278.8 -> 580.3 mm, vias 118 -> 137
- net KL30i: track 0.00 -> 186.6 mm, vias 0 -> 26
- net /Distance/SCL: track 8.83 -> 189.8 mm, vias 2 -> 15
- net /SigIn/~{RESET}: track 0.00 -> 171.7 mm, vias 0 -> 7
- net /Distance/SDA: track 24.8 -> 194.1 mm, vias 3 -> 15
- net /esp32s3/EN: track 0.00 -> 165.8 mm, vias 0 -> 5
- net /Speed/SCL_2: track 0.00 -> 141.5 mm, vias 0 -> 7
- net /BTN/BTN: track 8.00 -> 149.4 mm, vias 1 -> 6
- net /Speed/SDA_2: track 0.00 -> 135.9 mm, vias 0 -> 7
- net Net-(U101-~{OUT0}): track 145.4 -> 13.0 mm, vias 8 -> 1
- net /esp32s3/MOSI: track 0.00 -> 129.8 mm, vias 0 -> 3
- net /CAN/SCLK: track 0.00 -> 129.3 mm, vias 0 -> 3
- net /esp32s3/MISO: track 0.00 -> 128.6 mm, vias 0 -> 3
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- added copper zone on B.Cu, net /DC-DC/3V3_DCDC_Switch
- added copper zone on B.Cu, net /DC-DC/5V_DCDC_Switch
- added copper zone on B.Cu, net 3V3
- added copper zone on In2.Cu, net 3V3
- added copper zone on B.Cu, net KL30i
- removed copper zone on B.Cu, net (none)
- removed copper zone on In2.Cu, net (none)
Other:
- board text removed: "3V3"
- board text removed: "5V"
- board text removed: "KL30"
- board text removed: "KL31"

Commit message: maybe done?
Parts:
- added J2: Conn_01x08_Pin, Connector_Harwin:Harwin_M20-89008xx_1x08_P2.54mm_Horizontal, F.Cu at (120.5, -76.6)
Connections:
- U421 pad 2: 5V -> GND
- U601 pad 18: unconnected-(U601-IO10-Pad18) -> /esp32s3/LCD_DIN
- U601 pad 19: unconnected-(U601-IO11-Pad19) -> /esp32s3/LCD_CLK
- U601 pad 23: unconnected-(U601-IO21-Pad23) -> /esp32s3/LCD_DC
- U601 pad 24: unconnected-(U601-IO47-Pad24) -> /esp32s3/LCD_RST
- U601 pad 25: unconnected-(U601-IO48-Pad25) -> /esp32s3/LCD_CS
- U601 pad 26: unconnected-(U601-IO45-Pad26) -> /esp32s3/LCD_BLK
Routing:
- net /esp32s3/LCD_DIN: track 0.00 -> 15.0 mm, vias 0 -> 1
- net /esp32s3/LCD_CLK: track 0.00 -> 13.5 mm, vias 0 -> 1
- net /esp32s3/LCD_BLK: track 0.00 -> 13.3 mm, vias 0 -> 1
- net /esp32s3/LCD_RST: track 0.00 -> 12.7 mm, vias 0 -> 1
- net /esp32s3/LCD_DC: track 0.00 -> 11.6 mm, vias 0 -> 1
- net GND: track 580.3 -> 588.1 mm, vias 137 -> 139
- net /esp32s3/LCD_CS: track 0.00 -> 6.69 mm, vias 0 -> 1
- net 5V: track 214.0 -> 211.2 mm, vias 41 -> 39
- net /esp32s3/EN: track 165.8 -> 164.8 mm
- net /Distance/~{DIG-RST}: vias 21 -> 22
Other:
- board text added: "3V3"
- board text added: "5V"
- board text added: "5V GND DIN CLK CS DC RST BLK"
- board text added: "Speedometer RevB By Luca Bresch 03.12.2025"
