File: Speedometer/Speedometer_KiCAD_RevB/Hardware/Speedometer_Tech/Speedometer_Tech.kicad_pcb (KiCad board)
At the start: 4 copper layers, 309.2 x 103.7 mm, 239 parts, among them J1 Conn_01x03_Pin, J2 Conn_01x08_Pin, J800 776228-1, Q601 DTC123J, Q602 DTC123J, U1 MCP23017_SS, U100 TLC59108IPWR, U1001 TPS563200, U101 TLC59108IPWR, U1011 TPS563200, U102 TLC59108IPWR, U110 TLC59108IPWR, U111 TLC59108IPWR, U205 WS2812B-4020_2, U206 WS2812B-4020_2, U207 WS2812B-4020_2, U208 WS2812B-4020_2, U209 WS2812B-4020_2, U210 WS2812B-4020_2, U211 WS2812B-4020_2, U212 WS2812B-4020_2, U213 WS2812B-4020_2, U214 WS2812B-4020_2, U215 WS2812B-4020_2, U216 WS2812B-4020_2, U217 WS2812B-4020_2, U218 WS2812B-4020_2, U219 WS2812B-4020_2, U220 WS2812B-4020_2, U221 WS2812B-4020_2, U222 WS2812B-4020_2, U223 WS2812B-4020_2, U224 WS2812B-4020_2, U225 WS2812B-4020_2, U226 WS2812B-4020_2, U227 WS2812B-4020_2, U228 WS2812B-4020_2, U229 WS2812B-4020_2, U230 WS2812B-4020_2, U231 WS2812B-4020_2, U232 WS2812B-4020_2, U233 WS2812B-4020_2, U234 WS2812B-4020_2, U235 WS2812B-4020_2, U236 WS2812B-4020_2, U237 WS2812B-4020_2, U238 WS2812B-4020_2, U239 WS2812B-4020_2, U240 WS2812B-4020_2, U241 WS2812B-4020_2, U3 4010, U301 WS2812B-4020_2, U302 WS2812B-4020_2, U303 WS2812B-4020_2, U304 WS2812B-4020_2, U305 WS2812B-4020_2, U306 WS2812B-4020_2, U307 WS2812B-4020_2, U308 WS2812B-4020_2, U309 WS2812B-4020_2, U310 WS2812B-4020_2, U311 WS2812B-4020_2, U312 WS2812B-4020_2, U313 WS2812B-4020_2, U314 WS2812B-4020_2, U315 WS2812B-4020_2, U316 WS2812B-4020_2, U317 WS2812B-4020_2, U318 WS2812B-4020_2, U319 WS2812B-4020_2, U320 WS2812B-4020_2, U321 WS2812B-4020_2, U322 WS2812B-4020_2, U323 WS2812B-4020_2, U324 WS2812B-4020_2, U325 WS2812B-4020_2, U326 WS2812B-4020_2, U4 4010, U401 WS2812B-4020_2, U402 WS2812B-4020_2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

Commit message: pcb should be done now
Parts:
- added C1006: 22uF, Capacitor_SMD:C_0805_2012Metric, B.Cu at (137.0, -58.0)
- added C1016: 22uF, Capacitor_SMD:C_0805_2012Metric, B.Cu at (117.0, -57.5)
- added C604: 100nF, Capacitor_SMD:C_0603_1608Metric, B.Cu at (92.5, -83.0)
- added D1101: SBR80520LT1G, Diode_SMD:D_SOD-123, B.Cu at (27.5, -57.0)
- added D1102: SBR80520LT1G, Diode_SMD:D_SOD-123, B.Cu at (27.5, -53.6)
- added D1103: SBR80520LT1G, Diode_SMD:D_SOD-123, B.Cu at (27.5, -49.8)
- added D1104: SBR80520LT1G, Diode_SMD:D_SOD-123, B.Cu at (27.5, -46.5)
- moved C1014 1.51 mm to (114.0, -57.5)
- moved C1004 1.50 mm to (134.0, -58.0)
- moved C1005 1.50 mm to (131.0, -58.0)
- moved C1015 1.50 mm to (111.0, -57.5)
Routing:
- net 5V: track 211.2 -> 172.5 mm, vias 39 -> 37
- net VBUS: track 123.8 -> 146.0 mm
- net GND: track 588.1 -> 595.4 mm, vias 139 -> 142
- net KL30i: track 186.6 -> 193.5 mm
- net Net-(U603-VDD): track 0.00 -> 2.35 mm
- net 3V3: vias 24 -> 21

Commit message: Final Version, has been ordered
Parts:
- U605: moved to B.Cu
- moved R608 3.51 mm to (20.5, -50.0)
- moved R607 1.75 mm to (15.0, -53.0)
- turned U605 to -90 degrees
Routing:
- net GND: track 595.4 -> 593.5 mm
