File: Speedometer/Speedometer_KiCAD_RevB/Hardware/Speedometer_Tech/esp32S3.kicad_sch (KiCad schematic)
At the start: 31 parts, among them Q601 DTC123J, Q602 DTC123J, U601 ESP32-S3-WROOM-1(N8R2), U602 BC817, U603 CP2102N-A02-GQFN28R, U604 BC817, U605 YTC-TC16S-24, U606 TS35CA, U607 TS35CA

Commit message: Speedometer DRC mostly passed
Parts:
- removed U606, U607: TS35CA, footprint:KEY-SMD_TS35CA, symbol TS35CA:TS35CA
- added R611, R612: 2.2k, Resistor_SMD:R_0603_1608Metric, symbol AC0603DR-072K2L:AC0603DR-072K2L
- added S2, S606: SW_Omron_B3FS, Button_Switch_SMD:SW_SPST_Omron_B3FS-100xP, symbol Switch:SW_Omron_B3FS
- C601: footprint footprint:C0805 -> Capacitor_SMD:C_0805_2012Metric
- C602: footprint footprint:CAP-SMD_BD4.0-L4.3-W4.3-LS5.1-FD -> Capacitor_SMD:C_0805_2012Metric
- C603: footprint footprint:C0603 -> Capacitor_SMD:C_0201_0603Metric
- C605: footprint footprint:C0603 -> Resistor_SMD:R_0603_1608Metric
- H602: footprint footprint:HDR-TH_6P-P2.54-V-M-R2-C3-S2.54-1 -> Connector_PinHeader_2.54mm:PinHeader_2x03_P2.54mm_Vertical_SMD
- Q601, Q602: footprint (none) -> Package_TO_SOT_SMD:SOT-23
- R601, R602, R603, R604, R605, R606, R607, R608: footprint footprint:R0603 -> Resistor_SMD:R_0603_1608Metric
- R609, R610: footprint Resistor_SMD:R_0201_0603Metric -> Resistor_SMD:R_0603_1608Metric
- U602, U604: footprint footprint:SOT-23-3_L2.9-W1.3-P1.90-LS2.4-BR -> Package_TO_SOT_SMD:SOT-23-3
- U605: footprint footprint:USB-C-SMD_YTC-TC16S-24 -> Connector_USB:TYPEC-300D-BCP16H100
Connections:
- net BOOT: now also S606.2
- net EN: now also S2.2
- net GND: now also U605.A1 (GND), U605.A12 (GND), U605.B1 (GND), U605.B12 (GND), S2.1, S606.1; no longer U605.A12B1 (GND), U605.A1B12 (GND)
- net VBUS: now also U605.A4 (VBUS), U605.A9 (VBUS), U605.B4 (VBUS), U605.B9 (VBUS); no longer U605.A4B9 (VBUS), U605.A9B4 (VBUS)
- net ~{DIG-RST}: now also Q601.3 (C), R609.2
- net ~{RESET}: now also Q602.3 (C), R610.2
- net SDA_2: now reaches U601.13 (IO19)
- net SDA_2: now also R612.1
- net SCL_2: now reaches U601.14 (IO20)
- net SCL_2: now also R611.1
- net +3.3V renamed 3V3
- net 3V3: now also R611.2, R612.2
- no-connect marks 41 -> 39

Commit message: maybe done?
Parts:
- added J2: Conn_01x08_Pin, Connector_Harwin:Harwin_M20-89008xx_1x08_P2.54mm_Horizontal, symbol Connector:Conn_01x08_Pin
Connections:
- net 5V: now also J2.1 (Pin_1)
- net GND: now also J2.2 (Pin_2)
- net LCD_DIN: now reaches U601.18 (IO10)
- net LCD_DIN: now also J2.3 (Pin_3)
- net LCD_CLK: now reaches U601.19 (IO11)
- net LCD_CLK: now also J2.4 (Pin_4)
- net LCD_DC: now reaches U601.23 (IO21)
- net LCD_DC: now also J2.6 (Pin_6)
- net LCD_RST: now reaches U601.24 (IO47)
- net LCD_RST: now also J2.7 (Pin_7)
- net LCD_CS: now reaches U601.25 (IO48)
- net LCD_CS: now also J2.5 (Pin_5)
- net LCD_BLK: now reaches U601.26 (IO45)
- net LCD_BLK: now also J2.8 (Pin_8)
- no-connect marks 39 -> 33
Other:
- note added: "LCD Connector"

Commit message: pcb should be done now
Parts:
- removed D1101, D1102, D1103, D1104: SBR80520LT1G, FP-425-04-MFG, symbol Speedometer_Tech-altium-import:Designator_0_1d6ec82d83fb6aee721767c19dac4b9
- added D1101, D1102, D1103, D1104: SBR80520LT1G, Diode_SMD:D_SOD-123, symbol Device:D
- C604: footprint footprint:C0603 -> Capacitor_SMD:C_0603_1608Metric
Connections:
- net 5V: now also D1103.1 (K), D1104.1 (K)
- net KL30i: now also D1101.1 (K), D1102.1 (K)
- net VBUS: now also D1101.2 (A), D1102.2 (A), D1103.2 (A), D1104.2 (A)
